File: hardware/kicad/autofeeder.kicad_pcb (KiCad board)
At the start: 2 copper layers, 56 x 54 mm, 43 parts, among them J1 JST_XH_B2B-XH-A_1x02_P2.50mm_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, J2 JST_XH_B2B-XH-A_1x02_P2.50mm_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, J3 USB_C_Receptacle_HRO_TYPE-C-3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, J4 PinHeader_1x04_P2.54mm_Vertic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, SW1_POWER1 SW_Push_1P1T_NO_CK_KMR2, SW2_TIMER1 SW_Push_1P1T_NO_CK_KMR2, SW3_MANUAL1 SW_Push_1P1T_NO_CK_KMR2, SW4_SETTINGS1 SW_Push_1P1T_NO_CK_KMR2, SW5_UP1 SW_Push_1P1T_NO_CK_KMR2, SW6_DOWN1 SW_Push_1P1T_NO_CK_KMR2, U1 ESP32_C6_Zero, U2 SOIC-8_3.9x4.9mm_P1.27mm, U3 SOT-23-6_Handsoldering, U4 WSON-10-1EP_2.5x2.5mm_P0.5mm_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, U5 SOIC-8_3.9x4.9mm_P1.27mm, U6 SOIC-8_3.9x4.9mm_P1.27mm, U8 SOT-23-6_Handsoldering

Commit message: Fix BATT_N unconnected net, migrate to 4-layer PCB, refresh fab outputs
- Add _pre_route_batt_n() to route BATT_N net (DW01A ↔ FS8205A protection ICs)
  via B.Cu segments + F.Cu through-via, eliminating the last unconnected net
- Update README power topology to include DW01A/FS8205A protection
- Update docs/bom.md: 2→4 layer count, remove stale bodge wire instructions,
  update DRC status to reflect 0 unconnected items
- Regenerate all fab outputs (gerbers, drill, BOM, CPL, DRC) for 4-layer board
- Add inner copper layers (In1.Cu, In2.Cu) to gerber set
- Add Wabo Labs logo footprint, display_sleep custom component
- Add MX1508 reference datasheets
Parts:
- removed J2: JST_XH_B2B-XH-A_1x02_P2.50mm_Vertical, JST_XH_B2B-XH-A_1x02_P2.50mm_Vertical
- removed U5: SOIC-8_3.9x4.9mm_P1.27mm, SOIC-8_3.9x4.9mm_P1.27mm
- added J_MOTOR_CTRL1: JST_XH_B2B-XH-A_1x02_P2.50mm_Vertical, JST_XH_B2B-XH-A_1x02_P2.50mm_Vertical, B.Cu at (52.0, 14.0)
- added J_MOTOR_PWR1: JST_XH_B2B-XH-A_1x02_P2.50mm_Vertical, JST_XH_B2B-XH-A_1x02_P2.50mm_Vertical, B.Cu at (52.0, 24.0)
- added WABO_LOGO1: Wabo_Labs_Logo, Wabo_Labs_Logo, B.Cu at (30.0, 36.0)
- moved J_RTC1 15.2 mm to (42.0, 30.0)
- moved J1 4.00 mm to (52.0, 34.0)
- moved J4 2.00 mm to (53.0, 39.0)
Connections:
- U1 pad 22: unconnected-(U1-GP9/BOOT-Pad22) -> /CAN_RS
- U4 pad 11: (no net) -> GND
- U6 pad 8: /RS_NC -> /CAN_RS
Routing:
- net /M1_P: track 38.1 -> 0.00 mm, vias 1 -> 0
- net /M1_N: track 36.4 -> 0.00 mm, vias 1 -> 0
- net /VBUS: track 85.4 -> 49.6 mm, vias 2 -> 0
- net /L2_NODE: track 0.00 -> 33.2 mm
- net GND: track 308.6 -> 276.9 mm, vias 4 -> 249
- net /CC2: track 85.1 -> 55.9 mm, vias 0 -> 2
- net /CAN_RX: track 84.4 -> 56.4 mm, vias 0 -> 1
- net /L1_NODE: track 35.1 -> 14.1 mm
- net /CC1: track 67.0 -> 47.8 mm
- net /CAN_RS: track 0.00 -> 16.8 mm
- net /CAN_TX: track 63.9 -> 49.3 mm
- net /MOTOR_IN2: track 26.1 -> 40.0 mm
- net /MOTOR_IN1: track 25.8 -> 38.8 mm, vias 1 -> 0
- net /VCC_3V3: track 122.6 -> 133.4 mm, vias 1 -> 3
- net /BATT_P: track 69.3 -> 58.9 mm, vias 0 -> 1
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- added copper zone on In1.Cu, net GND
- added copper zone on In2.Cu, net GND
Other:
- copper layers 2 -> 4
- board text added: "CTRL"
- board text added: "PWR"
- board text removed: "MOTOR"
